Commit message: urdf

File: Robot_description/urdf/mid_tank_chassis.urdf (robot description, URDF)
Before this commit: robot mrobot_chassis, 2 links, 1 joints
Links:
- added link left_wheel_link; visual cylinder length=0.017 radius=0.033
Joints:
- added joint left_wheel_joint: type continuous, parent left_motor, child left_wheel_link, origin xyz=0 0.0485 0 rpy=0 0 0, axis 0 1 0
